Commit message: Fully modeled cutter

File: src/xarm_description/urdf/vader/vader_cutter.urdf.xacro (robot description, xacro)
@@ -2,12 +2,193 @@
 <robot xmlns:xacro="http://ros.org/wiki/xacro" name="vader_cutter">
   <xacro:macro name="vader_cutter_urdf" params="prefix:='' attach_to:='' attach_xyz:='0 0 0' attach_rpy:='0 0 0' ">
-    <xacro:unless value="${attach_to == ''}">
-      <joint name="${prefix}v_cutter_fix" type="fixed">
-        <parent link="${attach_to}"/>
-        <child link="${prefix}v_cutter_link"/>
-        <origin xyz="${attach_xyz}" rpy="${attach_rpy}"/>
-      </joint>
-    </xacro:unless>
-    <link name="${prefix}v_cutter_link">
+<!-- This URDF was automatically created by SolidWorks to URDF Exporter! Originally created by Stephen Brawner (brawner@gmail.com)
+     Commit Version: 1.6.0-4-g7f85cfe  Build Version: 1.6.7995.38578
+     For more information, please see http://wiki.ros.org/sw_urdf_exporter -->
+  <xacro:unless value="${attach_to == ''}">
+    <joint name="${prefix}v_cutter_fix" type="fixed">
+      <parent link="${attach_to}"/>
+      <child link="base_link"/>
+      <origin xyz="${attach_xyz}" rpy="${attach_rpy}"/>
+    </joint>
+  </xacro:unless>
+  <link
+    name="base_link">
+    <inertial>
+      <origin
+        xyz="0.000779839845872349 -0.0170873194546623 0.0582199927820382"
+        rpy="0 0 0" />
+      <mass
+        value="0.200722958769519" />
+      <inertia
+        ixx="0.000122002272224489"
+        ixy="-1.13774292063113E-06"
+        ixz="-4.83617188880724E-06"
+        iyy="0.000194887608314948"
+        iyz="2.99117381858236E-06"
+        izz="9.59225921675798E-05" />
+    </inertial>
+    <xacro:common_link_visual
+      mesh_filename="vader/cutter/base_link"
+      origin_xyz="0 0 0"
+      origin_rpy="0 0 0"
+      material_name="${prefix}White"/>
+    <xacro:common_link_collision
+      mesh_filename="vader/cutter/base_link"
+      origin_xyz="0 0 0"
+      origin_rpy="0 0 0" />
+    <!-- <visual>
+      <origin
+        xyz="0 0 0"
+        rpy="0 0 0" />
+      <geometry>
+        <mesh
+          filename="$(find xarm_description)/meshes/vader/cutter/base_link.stl" />
+      </geometry>
+      <material
+        name="">
+        <color
+          rgba="0.298039215686275 0.298039215686275 0.298039215686275 1" />
+      </material>
+    </visual>
+    <collision>
+      <origin
+        xyz="0 0 0"
+        rpy="0 0 0" />
+      <geometry>
+        <mesh
+          filename="$(find xarm_description)/meshes/vader/cutter/base_link.stl" />
+      </geometry>
+    </collision> -->
+  </link>
+  <link
+    name="blade_stationary">
+    <inertial>
+      <origin
+        xyz="-0.00557368894630381 -0.0122907539881133 0.00132925858009713"
+        rpy="0 0 0" />
+      <mass
+        value="0.0157008165066123" />
+      <inertia
+        ixx="3.54894565615037E-06"
+        ixy="-1.00617922467536E-06"
+        ixz="4.9211811874153E-09"
+        iyy="1.01338167968976E-06"
+        iyz="4.1050442824912E-08"
+        izz="4.54778499319921E-06" />
+    </inertial>
+    <!-- <visual>
+      <origin
+        xyz="0 0 0"
+        rpy="0 0 0" />
+      <geometry>
+        <mesh
+          filename="$(find xarm_description)/meshes/vader/cutter/blade_stationary.stl" />
+      </geometry>
+      <material
+        name="">
+        <color
+          rgba="0.898039215686275 0.898039215686275 0.898039215686275 1" />
+      </material>
+    </visual>
+    <collision>
+      <origin
+        xyz="0 0 0"
+        rpy="0 0 0" />
+      <geometry>
+        <mesh
+          filename="$(find xarm_description)/meshes/vader/cutter/blade_stationary.stl" />
+      </geometry>
+    </collision> -->
+    <xacro:common_link_visual
+      mesh_filename="vader/cutter/blade_stationary"
+      origin_xyz="0 0 0"
+      origin_rpy="0 0 0"
+      material_name="${prefix}White"/>
+    <xacro:common_link_collision
+      mesh_filename="vader/cutter/blade_stationary"
+      origin_xyz="0 0 0"
+      origin_rpy="0 0 0" />
+  </link>
+  <joint
+    name="joint_blade_stationary"
+    type="fixed">
+    <origin
+      xyz="0 -0.0083875 0.12394"
+      rpy="-1.5708 0 0" />
+    <parent
+      link="base_link" />
+    <child
+      link="blade_stationary" />
+    <axis
+      xyz="0 0 0" />
+  </joint>
+  <link
+    name="blade_moving">
+    <inertial>
+      <origin
+        xyz="3.87969033185664E-05 -0.00350154660982081 0.00219998568406248"
+        rpy="0 0 0" />
+      <mass
+        value="0.0382144342405943" />
+      <inertia
+        ixx="8.88222836308347E-06"
+        ixy="7.69834936555405E-06"
+        ixz="4.74020773662496E-12"
+        iyy="1.00340865289331E-05"
+        iyz="1.44904462744025E-11"
+        izz="1.87930181166959E-05" />
+    </inertial>
+    <!-- <visual>
+      <origin
+        xyz="0 0 0"
+        rpy="0 0 0" />
+      <geometry>
+        <mesh
+          filename="$(find xarm_description)/meshes/vader/cutter/blade_moving.stl" />
+      </geometry>
+      <material
+        name="">
+        <color
+          rgba="0.776470588235294 0.756862745098039 0.737254901960784 1" />
+      </material>
+    </visual>
+    <collision>
+      <origin
+        xyz="0 0 0"
+        rpy="0 0 0" />
+      <geometry>
+        <mesh
+          filename="$(find xarm_description)/meshes/vader/cutter/blade_moving.stl" />
+      </geometry>
+    </collision> -->
+    <xacro:common_link_visual
+      mesh_filename="vader/cutter/blade_moving"
+      origin_xyz="0 0 0"
+      origin_rpy="0 0 0"
+      material_name="${prefix}White"/>
+    <xacro:common_link_collision
+      mesh_filename="vader/cutter/blade_moving"
+      origin_xyz="0 0 0"
+      origin_rpy="0 0 0" />
+  </link>
+  <joint
+    name="joint_blade"
+    type="revolute">
+    <origin
+      xyz="0 -0.0059875 0.12394"
+      rpy="-1.5708 0 0" />
+    <parent
+      link="base_link" />
+    <child
+      link="blade_moving" />
+    <limit
+      effort="0.5"
+      lower="-3.14159265358979"
+      upper="3.14159265358979"
+      velocity="1" />
+    <axis
+      xyz="0 0 1" />
+  </joint>
+    <!-- <link name="base_link">
       <inertial>
         <origin xyz="0.0 0.0 0.055" rpy="0 0 0" />
@@ -26,10 +207,10 @@
         origin_xyz="0 0 0"
         origin_rpy="0 0 0" />
-    </link>
+    </link> -->
     <!-- TODO add actual URDF -->
     <link name="${prefix}link_tcp" />
     <joint name="${prefix}joint_tcp" type="fixed">
       <origin xyz="0 0 0.126" rpy="0 0 0" />
-      <parent link="${prefix}v_cutter_link" />
+      <parent link="base_link" />
       <child link="${prefix}link_tcp" />
     </joint>

Commit message: Updated cutter xacro, completed gripper xacro. Both have full mesh but not controllable yet

File: src/xarm_description/urdf/vader/vader_cutter.urdf.xacro (robot description, xacro)
@@ -2,7 +2,4 @@
 <robot xmlns:xacro="http://ros.org/wiki/xacro" name="vader_cutter">
   <xacro:macro name="vader_cutter_urdf" params="prefix:='' attach_to:='' attach_xyz:='0 0 0' attach_rpy:='0 0 0' ">
-<!-- This URDF was automatically created by SolidWorks to URDF Exporter! Originally created by Stephen Brawner (brawner@gmail.com)
-     Commit Version: 1.6.0-4-g7f85cfe  Build Version: 1.6.7995.38578
-     For more information, please see http://wiki.ros.org/sw_urdf_exporter -->
   <xacro:unless value="${attach_to == ''}">
     <joint name="${prefix}v_cutter_fix" type="fixed">

File: src/xarm_description/urdf/vader/vader_gripper.urdf.xacro (robot description, xacro)
@@ -1,13 +1,14 @@
 <?xml version="1.0"?>
 <robot xmlns:xacro="http://ros.org/wiki/xacro" name="vader_gripper">
-  <xacro:macro name="vader_gripper_urdf" params="prefix:='' attach_to:='' attach_xyz:='0 0 0' attach_rpy:='0 0 0' ">
+  <xacro:macro name="vader_gripper_urdf" params="prefix:='' attach_to:='' attach_xyz:='0 0 0.0795' attach_rpy:='0 0 0' ">
     <xacro:unless value="${attach_to == ''}">
       <joint name="${prefix}v_gripper_fix" type="fixed">
         <parent link="${attach_to}"/>
-        <child link="${prefix}v_gripper_link"/>
+        <child link="base_link"/>
         <origin xyz="${attach_xyz}" rpy="${attach_rpy}"/>
       </joint>
     </xacro:unless>
-    <link name="${prefix}v_gripper_link">
+<!--
+    <link name="base_link">
       <inertial>
         <origin xyz="0.0 0.0 0.055" rpy="0 0 0" />
@@ -26,10 +27,259 @@
         origin_xyz="0 0 0"
         origin_rpy="0 0 0" />
-    </link>
-    <!-- TODO add actual URDF -->
+    </link> -->
+  <link
+    name="base_link">
+    <inertial>
+      <origin
+        xyz="-9.9221E-05 -0.0018613 -0.03661"
+        rpy="0 0 0" />
+      <mass
+        value="0.28958" />
+      <inertia
+        ixx="0.00019685"
+        ixy="2.3047E-07"
+        ixz="-6.0829E-07"
+        iyy="0.00010064"
+        iyz="7.7606E-07"
+        izz="0.00023082" />
+    </inertial>
+    <!-- <visual>
+      <origin
+        xyz="0 0 0"
+        rpy="0 0 0" />
+      <geometry>
+        <mesh
+          filename="package://gripper/meshes/base_link.STL" />
+      </geometry>
+      <material
+        name="">
+        <color
+          rgba="0.79216 0.81961 0.93333 1" />
+      </material>
+    </visual>
+    <collision>
+      <origin
+        xyz="0 0 0"
+        rpy="0 0 0" />
+      <geometry>
+        <mesh
+          filename="package://gripper/meshes/base_link.STL" />
+      </geometry>
+    </collision> -->
+    <xacro:common_link_visual
+      mesh_filename="vader/gripper/base_link"
+      origin_xyz="0 0 0"
+      origin_rpy="0 0 0"
+      material_name="${prefix}White"/>
+    <xacro:common_link_collision
+      mesh_filename="vader/gripper/base_link"
+      origin_xyz="0 0 0"
+      origin_rpy="0 0 0" />
+  </link>
+  <link
+    name="thumb_1">
+    <inertial>
+      <origin
+        xyz="2.6455E-07 0.043188 -0.043887"
+        rpy="0 0 0" />
+      <mass
+        value="0.037019" />
+      <inertia
+        ixx="5.4009E-06"
+        ixy="1.033E-11"
+        ixz="1.696E-11"
+        iyy="4.3501E-06"
+        iyz="1.9961E-06"
+        izz="4.1256E-06" />
+    </inertial>
+    <!-- <visual>
+      <origin
+        xyz="0 0 0"
+        rpy="0 0 0" />
+      <geometry>
+        <mesh
+          filename="package://gripper/meshes/thumb_1.STL" />
+      </geometry>
+      <material
+        name="">
+        <color
+          rgba="0.79216 0.81961 0.93333 1" />
+      </material>
+    </visual>
+    <collision>
+      <origin
+        xyz="0 0 0"
+        rpy="0 0 0" />
+      <geometry>
+        <mesh
+          filename="package://gripper/meshes/thumb_1.STL" />
+      </geometry>
+    </collision> -->
+    <xacro:common_link_visual
+      mesh_filename="vader/gripper/thumb_1"
+      origin_xyz="0 0 0"
+      origin_rpy="0 0 0"
+      material_name="${prefix}White"/>
+    <xacro:common_link_collision
+      mesh_filename="vader/gripper/thumb_1"
+      origin_xyz="0 0 0"
+      origin_rpy="0 0 0" />
+  </link>
+  <joint
+    name="thumb_joint"
+    type="revolute">
+    <origin
+      xyz="0 0.045195 0.013956"
+      rpy="2.7397 0 -3.1416" />
+    <parent
+      link="base_link" />
+    <child
+      link="thumb_1" />
+    <axis
+      xyz="-1 0 0" />
+    <limit
+      lower="0"
+      upper="0"
+      effort="0"
+      velocity="0" />
+  </joint>
+  <link
+    name="fing_1">
+    <inertial>
+      <origin
+        xyz="4.6591E-08 0.0003852 0.045879"
+        rpy="0 0 0" />
+      <mass
+        value="0.023872" />
+      <inertia
+        ixx="2.3287E-06"
+        ixy="-3.8578E-12"
+        ixz="1.8688E-12"
+        iyy="3.018E-06"
+        iyz="-9.0604E-08"
+        izz="1.2808E-06" />
+    </inertial>
+    <!-- <visual>
+      <origin
+        xyz="0 0 0"
+        rpy="0 0 0" />
+      <geometry>
+        <mesh
+          filename="package://gripper/meshes/fing_1.STL" />
+      </geometry>
+      <material
+        name="">
+        <color
+          rgba="0.79216 0.81961 0.93333 1" />
+      </material>
+    </visual>
+    <collision>
+      <origin
+        xyz="0 0 0"
+        rpy="0 0 0" />
+      <geometry>
+        <mesh
+          filename="package://gripper/meshes/fing_1.STL" />
+      </geometry>
+    </collision> -->
+    <xacro:common_link_visual
+      mesh_filename="vader/gripper/fing_1"
+      origin_xyz="0 0 0"
+      origin_rpy="0 0 0"
+      material_name="${prefix}White"/>
+    <xacro:common_link_collision
+      mesh_filename="vader/gripper/fing_1"
+      origin_xyz="0 0 0"
+      origin_rpy="0 0 0" />
+  </link>
+  <joint
+    name="fing_1_joint"
+    type="revolute">
+    <origin
+      xyz="0.018 -0.045195 0.013956"
+      rpy="0.40187 0 0" />
+    <parent
+      link="base_link" />
+    <child
+      link="fing_1" />
+    <axis
+      xyz="-1 0 0" />
+    <limit
+      lower="0"
+      upper="0"
+      effort="0"
+      velocity="0" />
+  </joint>
+  <link
+    name="fing_2">
+    <inertial>
+      <origin
+        xyz="4.7008E-08 0.0003852 0.045879"
+        rpy="0 0 0" />
+      <mass
+        value="0.023872" />
+      <inertia
+        ixx="2.3287E-06"
+        ixy="-3.9096E-12"
+        ixz="1.8436E-12"
+        iyy="3.018E-06"
+        iyz="-9.0604E-08"
+        izz="1.2808E-06" />
+    </inertial>
+    <!-- <visual>
+      <origin
+        xyz="0 0 0"
+        rpy="0 0 0" />
+      <geometry>
+        <mesh
+          filename="package://gripper/meshes/fing_2.STL" />
+      </geometry>
+      <material
+        name="">
+        <color
+          rgba="0.79216 0.81961 0.93333 1" />
+      </material>
+    </visual>
+    <collision>
+      <origin
+        xyz="0 0 0"
+        rpy="0 0 0" />
+      <geometry>
+        <mesh
+          filename="package://gripper/meshes/fing_2.STL" />
+      </geometry>
+    </collision> -->
+    <xacro:common_link_visual
+      mesh_filename="vader/gripper/fing_2"
+      origin_xyz="0 0 0"
+      origin_rpy="0 0 0"
+      material_name="${prefix}White"/>
+    <xacro:common_link_collision
+      mesh_filename="vader/gripper/fing_2"
+      origin_xyz="0 0 0"
+      origin_rpy="0 0 0" />
+  </link>
+  <joint
+    name="fing_2_joint"
+    type="revolute">
+    <origin
+      xyz="-0.018 -0.045195 0.013956"
+      rpy="0.40187 0 0" />
+    <parent
+      link="base_link" />
+    <child
+      link="fing_2" />
+    <axis
+      xyz="-1 0 0" />
+    <limit
+      lower="0"
+      upper="0"
+      effort="0"
+      velocity="0" />
+  </joint>
     <link name="${prefix}link_tcp" />
     <joint name="${prefix}joint_tcp" type="fixed">
       <origin xyz="0 0 0.126" rpy="0 0 0" />
-      <parent link="${prefix}v_gripper_link" />
+      <parent link="base_link" />
       <child link="${prefix}link_tcp" />
     </joint>

Commit message: WIP completed gazebo and transmission files, need to test

File: src/xarm_description/urdf/vader/vader_cutter.urdf.xacro (robot description, xacro)
@@ -5,10 +5,10 @@
     <joint name="${prefix}v_cutter_fix" type="fixed">
       <parent link="${attach_to}"/>
-      <child link="base_link"/>
+      <child link="vader_cutter_base_link"/>
       <origin xyz="${attach_xyz}" rpy="${attach_rpy}"/>
     </joint>
   </xacro:unless>
   <link
-    name="base_link">
+    name="vader_cutter_base_link">
     <inertial>
       <origin
@@ -114,5 +114,5 @@
       rpy="-1.5708 0 0" />
     <parent
-      link="base_link" />
+      link="vader_cutter_base_link" />
     <child
       link="blade_stationary" />
@@ -176,5 +176,5 @@
       rpy="-1.5708 0 0" />
     <parent
-      link="base_link" />
+      link="vader_cutter_base_link" />
     <child
       link="blade_moving" />
@@ -187,5 +187,5 @@
       xyz="0 0 1" />
   </joint>
-    <!-- <link name="base_link">
+    <!-- <link name="vader_cutter_base_link">
       <inertial>
         <origin xyz="0.0 0.0 0.055" rpy="0 0 0" />
@@ -209,5 +209,5 @@
     <joint name="${prefix}joint_tcp" type="fixed">
       <origin xyz="0 0 0.126" rpy="0 0 0" />
-      <parent link="base_link" />
+      <parent link="vader_cutter_base_link" />
       <child link="${prefix}link_tcp" />
     </joint>

File: src/xarm_description/urdf/vader/vader_cutter_macro.xacro (robot description, xacro)
@@ -1,4 +1,8 @@
 <?xml version='1.0' encoding='utf-8'?>
 <robot xmlns:xacro="http://ros.org/wiki/xacro" name="vader_cutter">
+  <!-- imports -->
+  <xacro:include filename="$(find xarm_description)/urdf/vader/vader_cutter.urdf.xacro" />
+  <xacro:include filename="$(find xarm_description)/urdf/vader/vader_cutter.transmission.xacro" />
+  <xacro:include filename="$(find xarm_description)/urdf/vader/vader_cutter.gazebo.xacro" />
   <xacro:macro name="vader_cutter_macro" params="prefix:='' attach_to:='' robot_type:='xarm' mesh_suffix:='stl' hard_interface:='' ">
     <!-- Load Common Material -->
@@ -14,4 +18,14 @@
     <xacro:include filename="$(find xarm_description)/urdf/vader/vader_cutter.urdf.xacro" />
     <xacro:vader_cutter_urdf prefix="${prefix}" attach_to="${attach_to}"/>
+    <!-- Sim items -->
+    <xacro:vader_cutter_transmission prefix="${prefix}" hard_interface="${hard_interface}" />
+    <xacro:vader_cutter_gazebo prefix="${prefix}" />
+    <xacro:vader_cutter_grasp_fix prefix="${prefix}" palm_link="${prefix}link${dof}" />
+    <xacro:mimic_joint_plugin_gazebo name_prefix="vader_cutter_fing_1_mimic"
+      following_joint="thumb_joint" mimic_joint="fing_1_joint"
+      has_pid="false" multiplier="1.0" max_effort="10.0" />
+    <xacro:mimic_joint_plugin_gazebo name_prefix="vader_cutter_fing_2_mimic"
+      following_joint="thumb_joint" mimic_joint="fing_2_joint"
+      has_pid="false" multiplier="1.0" max_effort="10.0" />
   </xacro:macro>
 </robot>

File: src/xarm_description/urdf/vader/vader_gripper.urdf.xacro (robot description, xacro)
@@ -5,10 +5,10 @@
       <joint name="${prefix}v_gripper_fix" type="fixed">
         <parent link="${attach_to}"/>
-        <child link="base_link"/>
+        <child link="vader_gripper_base_link"/>
         <origin xyz="${attach_xyz}" rpy="${attach_rpy}"/>
       </joint>
     </xacro:unless>
 <!--
-    <link name="base_link">
+    <link name="vader_gripper_base_link">
       <inertial>
         <origin xyz="0.0 0.0 0.055" rpy="0 0 0" />
@@ -29,5 +29,5 @@
     </link> -->
   <link
-    name="base_link">
+    name="vader_gripper_base_link">
     <inertial>
       <origin
@@ -133,5 +133,5 @@
       rpy="2.7397 0 -3.1416" />
     <parent
-      link="base_link" />
+      link="vader_gripper_base_link" />
     <child
       link="thumb_1" />
@@ -200,5 +200,5 @@
       rpy="0.40187 0 0" />
     <parent
-      link="base_link" />
+      link="vader_gripper_base_link" />
     <child
       link="fing_1" />
@@ -267,5 +267,5 @@
       rpy="0.40187 0 0" />
     <parent
-      link="base_link" />
+      link="vader_gripper_base_link" />
     <child
       link="fing_2" />
@@ -281,5 +281,5 @@
     <joint name="${prefix}joint_tcp" type="fixed">
       <origin xyz="0 0 0.126" rpy="0 0 0" />
-      <parent link="base_link" />
+      <parent link="vader_gripper_base_link" />
       <child link="${prefix}link_tcp" />
     </joint>

File: src/xarm_description/urdf/vader/vader_gripper_macro.xacro (robot description, xacro)
@@ -1,4 +1,8 @@
 <?xml version='1.0' encoding='utf-8'?>
 <robot xmlns:xacro="http://ros.org/wiki/xacro" name="vader_gripper">
+  <!-- imports -->
+  <xacro:include filename="$(find xarm_description)/urdf/vader/vader_gripper.urdf.xacro" />
+  <xacro:include filename="$(find xarm_description)/urdf/vader/vader_gripper.transmission.xacro" />
+  <xacro:include filename="$(find xarm_description)/urdf/vader/vader_gripper.gazebo.xacro" />
   <xacro:macro name="vader_gripper_macro" params="prefix:='' attach_to:='' robot_type:='xarm' mesh_suffix:='stl' hard_interface:='' ">
     <!-- Load Common Material -->
@@ -14,4 +18,12 @@
     <xacro:include filename="$(find xarm_description)/urdf/vader/vader_gripper.urdf.xacro" />
     <xacro:vader_gripper_urdf prefix="${prefix}" attach_to="${attach_to}"/>
+    <!-- Sim items -->
+    <xacro:vader_gripper_transmission prefix="${prefix}" hard_interface="${hard_interface}" />
+    <xacro:vader_gripper_gazebo prefix="${prefix}" />
+    <xacro:vader_gripper_grasp_fix prefix="${prefix}" palm_link="${prefix}link${dof}" />
+    <!-- mimic_joint_plugin has to be installed: -->
+    <xacro:mimic_joint_plugin_gazebo name_prefix="${prefix}bio_gripper_left_finger_joint"
+      following_joint="${prefix}right_finger_joint" mimic_joint="${prefix}left_finger_joint"
+      has_pid="false" multiplier="-1.0" max_effort="10.0" />
   </xacro:macro>
 </robot>
