Commit message: Fully functional gripper fingers as three separate joints, since mimic plugin is not functional

File: src/xarm_description/urdf/vader/vader_cutter_macro.xacro (robot description, xacro)
@@ -22,10 +22,4 @@
     <xacro:vader_cutter_gazebo prefix="${prefix}" />
     <xacro:vader_cutter_grasp_fix prefix="${prefix}" palm_link="${prefix}link${dof}" />
-    <xacro:mimic_joint_plugin_gazebo name_prefix="vader_cutter_fing_1_mimic"
-      following_joint="thumb_joint" mimic_joint="fing_1_joint"
-      has_pid="false" multiplier="1.0" max_effort="10.0" />
-    <xacro:mimic_joint_plugin_gazebo name_prefix="vader_cutter_fing_2_mimic"
-      following_joint="thumb_joint" mimic_joint="fing_2_joint"
-      has_pid="false" multiplier="1.0" max_effort="10.0" />
   </xacro:macro>
 </robot>

File: src/xarm_description/urdf/vader/vader_gripper.transmission.xacro (robot description, xacro)
@@ -3,10 +3,30 @@
   <xacro:macro name="vader_gripper_transmission"
     params="prefix hard_interface:=PositionJointInterface reduction:=1">
-    <transmission name="${prefix}vader_gripper_joint_trans">
+    <transmission name="${prefix}vader_gripper_t_joint_trans">
       <type>transmission_interface/SimpleTransmission</type>
+      <actuator name="thumb_joint_motor">
+        <hardwareInterface>hardware_interface/${hard_interface}</hardwareInterface>
+        <mechanicalReduction>${reduction}</mechanicalReduction>
+      </actuator>
       <joint name="thumb_joint">
         <hardwareInterface>hardware_interface/${hard_interface}</hardwareInterface>
       </joint>
-      <actuator name="thumb_joint_motor">
+      </transmission>
+    <transmission name="${prefix}vader_gripper_1_joint_trans">
+      <type>transmission_interface/SimpleTransmission</type>
+      <joint name="fing_1_joint">
+        <hardwareInterface>hardware_interface/${hard_interface}</hardwareInterface>
+      </joint>
+      <actuator name="fing_1_joint_motor">
+        <hardwareInterface>hardware_interface/${hard_interface}</hardwareInterface>
+        <mechanicalReduction>${reduction}</mechanicalReduction>
+      </actuator>
+      </transmission>
+    <transmission name="${prefix}vader_gripper_2_joint_trans">
+      <type>transmission_interface/SimpleTransmission</type>
+      <joint name="fing_2_joint">
+        <hardwareInterface>hardware_interface/${hard_interface}</hardwareInterface>
+      </joint>
+      <actuator name="fing_2_joint_motor">
         <hardwareInterface>hardware_interface/${hard_interface}</hardwareInterface>
         <mechanicalReduction>${reduction}</mechanicalReduction>

File: src/xarm_description/urdf/vader/vader_gripper_macro.xacro (robot description, xacro)
@@ -23,7 +23,16 @@
     <xacro:vader_gripper_grasp_fix prefix="${prefix}" palm_link="${prefix}link${dof}" />
     <!-- mimic_joint_plugin has to be installed: -->
-    <xacro:mimic_joint_plugin_gazebo name_prefix="${prefix}bio_gripper_left_finger_joint"
-      following_joint="${prefix}right_finger_joint" mimic_joint="${prefix}left_finger_joint"
-      has_pid="false" multiplier="-1.0" max_effort="10.0" />
+    <!-- <xacro:mimic_joint_plugin_gazebo name_prefix="vader_cutter_fing_1_mimic"
+      following_joint="thumb_joint" mimic_joint="fing_1_joint"
+      has_pid="false" multiplier="1.0" max_effort="10.0" />
+    <xacro:mimic_joint_plugin_gazebo name_prefix="vader_cutter_fing_2_mimic"
+      following_joint="thumb_joint" mimic_joint="fing_2_joint"
+      has_pid="false" multiplier="1.0" max_effort="10.0" /> -->
+    <!-- <xacro:mimic_joint_plugin_gazebo name_prefix="vg_mimic_1_"
+      following_joint="thumb_joint" mimic_joint="fing_1_joint"
+      has_pid="true" multiplier="1.0" max_effort="10.0" />
+    <xacro:mimic_joint_plugin_gazebo name_prefix="vg_mimic_2_"
+      following_joint="thumb_joint" mimic_joint="fing_2_joint"
+      has_pid="true" multiplier="1.0" max_effort="10.0" /> -->
   </xacro:macro>
 </robot>
