Commit message: Pepper breakable with breakable joints plugin, demo world uploaded, xarm_controller beefed up to generate greater force

File: src/xarm_description/urdf/vader/vader_cutter.gazebo.xacro (robot description, xacro)
@@ -22,4 +22,5 @@
     </gazebo>
   </xacro:macro>
+<!--
   <xacro:macro name="vader_cutter_grasp_fix" params="prefix:='' arm_name:='vader_gripper' palm_link:=''">
     <gazebo>
@@ -40,5 +41,5 @@
       </plugin>
     </gazebo>
-  </xacro:macro>
+  </xacro:macro> -->
   <xacro:macro name="vader_cutter_gazebo" params="prefix">
     <gazebo reference="vader_cutter_base_link">

File: src/xarm_description/urdf/vader/vader_cutter.urdf.xacro (robot description, xacro)
@@ -180,8 +180,8 @@
       link="blade_moving" />
     <limit
-      effort="0.5"
+      effort="5"
       lower="-0.75"
       upper="0"
-      velocity="1" />
+      velocity="100" />
     <axis
       xyz="0 0 1" />

File: src/xarm_description/urdf/vader/vader_cutter_macro.xacro (robot description, xacro)
@@ -21,5 +21,5 @@
     <xacro:vader_cutter_transmission prefix="${prefix}" hard_interface="${hard_interface}" />
     <xacro:vader_cutter_gazebo prefix="${prefix}" />
-    <xacro:vader_cutter_grasp_fix prefix="${prefix}" palm_link="${prefix}link${dof}" />
+    <!-- <xacro:vader_cutter_grasp_fix prefix="${prefix}" palm_link="${prefix}link${dof}" /> -->
   </xacro:macro>
 </robot>
