Commit message: Added submodules for missing gazebo grasp fix plugin, pepper is now able to be grasped and released

File: src/xarm_description/urdf/vader/vader_gripper.gazebo.xacro (robot description, xacro)
@@ -21,5 +21,5 @@
     </gazebo>
   </xacro:macro>
-  <xacro:macro name="vader_gripper_grasp_fix" params="prefix:='' arm_name:='xarm_gripper' palm_link:='link_base'">
+  <xacro:macro name="vader_gripper_grasp_fix" params="prefix:='' arm_name:='xarm' palm_link:='link_base'">
     <gazebo>
       <plugin name="gazebo_grasp_fix" filename="libgazebo_grasp_fix.so">
@@ -35,5 +35,5 @@
         <grip_count_threshold>2</grip_count_threshold>
         <max_grip_count>3</max_grip_count>
-        <release_tolerance>0.0198</release_tolerance>
+        <release_tolerance>0.005</release_tolerance>
         <disable_collisions_on_attach>false</disable_collisions_on_attach>
         <contact_topic>__default_topic__</contact_topic>

File: src/xarm_description/urdf/vader/vader_gripper.urdf.xacro (robot description, xacro)
@@ -141,5 +141,5 @@
       lower="-1"
       upper="1.5"
-      effort="1" velocity="1" />
+      effort="5" velocity="1" />
   </joint>
   <link
@@ -207,5 +207,5 @@
       lower="-1"
       upper="1.5"
-      effort="1" velocity="1" />
+      effort="5" velocity="1" />
   </joint>
   <link
@@ -273,5 +273,5 @@
       lower="-1"
       upper="1.5"
-      effort="1" velocity="1" />
+      effort="5" velocity="1" />
   </joint>
     <link name="${prefix}link_tcp" />
