Commit message: Added SRDF and tweaks. Collision checking is configured and arms with end effectors can now be used with MoveIt

File: src/xarm_description/srdf/_xarm7_macro.srdf.xacro (robot description, xacro)
@@ -10,5 +10,5 @@
   <!-- SUBGROUPS: Groups can also be formed by referencing to already defined group names -->
   <xacro:macro name="xarm7_macro_srdf" params="prefix=''
-    add_gripper='false' add_vacuum_gripper='false' add_other_geometry='false' ">
+    add_gripper='false' add_vader_gripper='false' add_vader_cutter='false' add_vacuum_gripper='false' add_other_geometry='false' ">
     <xacro:if value="${add_gripper}">
       <xacro:property name="_use_gripper" value="true"/>
@@ -16,4 +16,6 @@
       <xacro:property name="_use_other_geometry" value="false"/>
       <xacro:property name="_use_no_end_effector" value="false"/>
+      <xacro:property name="_use_vader_gripper" value="false"/>
+      <xacro:property name="_use_vader_cutter" value="false"/>
     </xacro:if>
     <xacro:unless value="${add_gripper}">
@@ -23,4 +25,6 @@
         <xacro:property name="_use_other_geometry" value="false"/>
         <xacro:property name="_use_no_end_effector" value="false"/>
+        <xacro:property name="_use_vader_gripper" value="false"/>
+        <xacro:property name="_use_vader_cutter" value="false"/>
       </xacro:if>
       <xacro:unless value="${add_vacuum_gripper}">
@@ -30,10 +34,34 @@
           <xacro:property name="_use_other_geometry" value="true"/>
           <xacro:property name="_use_no_end_effector" value="false"/>
+          <xacro:property name="_use_vader_gripper" value="false"/>
+          <xacro:property name="_use_vader_cutter" value="false"/>
         </xacro:if>
         <xacro:unless value="${add_other_geometry}">
-          <xacro:property name="_use_gripper" value="false"/>
-          <xacro:property name="_use_vacuum_gripper" value="false"/>
-          <xacro:property name="_use_other_geometry" value="false"/>
-          <xacro:property name="_use_no_end_effector" value="true"/>
+          <xacro:if value="${add_vader_gripper}">
+            <xacro:property name="_use_gripper" value="false"/>
+            <xacro:property name="_use_vacuum_gripper" value="false"/>
+            <xacro:property name="_use_other_geometry" value="false"/>
+            <xacro:property name="_use_no_end_effector" value="false"/>
+            <xacro:property name="_use_vader_gripper" value="true"/>
+            <xacro:property name="_use_vader_cutter" value="false"/>
+          </xacro:if>
+          <xacro:unless value="${add_vader_gripper}">
+            <xacro:if value="${add_vader_cutter}">
+              <xacro:property name="_use_gripper" value="false"/>
+              <xacro:property name="_use_vacuum_gripper" value="false"/>
+              <xacro:property name="_use_other_geometry" value="false"/>
+              <xacro:property name="_use_no_end_effector" value="false"/>
+              <xacro:property name="_use_vader_gripper" value="false"/>
+              <xacro:property name="_use_vader_cutter" value="true"/>
+            </xacro:if>
+            <xacro:unless value="${add_vader_cutter}"> <!--no EEF-->
+              <xacro:property name="_use_gripper" value="false"/>
+              <xacro:property name="_use_vacuum_gripper" value="false"/>
+              <xacro:property name="_use_other_geometry" value="false"/>
+              <xacro:property name="_use_no_end_effector" value="true"/>
+              <xacro:property name="_use_vader_gripper" value="true"/>
+              <xacro:property name="_use_vader_cutter" value="false"/>
+            </xacro:unless>
+          </xacro:unless>
         </xacro:unless>
       </xacro:unless>
@@ -51,4 +79,12 @@
       <xacro:if value="${_use_gripper}">
         <joint name="${prefix}gripper_fix" />
+        <joint name="${prefix}joint_tcp" />
+      </xacro:if>
+      <xacro:if value="${_use_vader_gripper}">
+        <!-- <joint name="vader_gripper_grasp_fix" /> -->
+        <joint name="${prefix}joint_tcp" />
+      </xacro:if>
+      <xacro:if value="${_use_vader_cutter}">
+        <!-- <joint name="vader_cutter_grasp_fix" /> -->
         <joint name="${prefix}joint_tcp" />
       </xacro:if>
@@ -182,4 +218,45 @@
       <disable_collisions link1="${prefix}link_eef" link2="${prefix}xarm_vacuum_gripper_link" reason="Adjacent" />
     </xacro:if>
+    <!-- vader gripper -->
+    <xacro:if value="${_use_vader_gripper}">
+      <group name="${prefix}vader_gripper">
+        <!-- <joint name="${prefix}v_gripper_fix" /> -->
+        <link name="fing_1" />
+        <link name="fing_2" />
+        <link name="thumb_1" />
+        <link name="${prefix}link_tcp" />
+        <link name="vader_gripper_base_link"/>
+      </group>
+      <end_effector name="${prefix}vader_gripper" parent_link="${prefix}link_tcp" group="${prefix}vader_gripper" />
+      <!-- <passive_joint name="${prefix}v_gripper_fix" /> -->
+      <!-- <disable_collisions link1="${prefix}link3" link2="" reason="Never" />
+      <disable_collisions link1="${prefix}link6" link2="${prefix}xarm_vacuum_gripper_link" reason="Never" />
+      <disable_collisions link1="${prefix}link7" link2="${prefix}xarm_vacuum_gripper_link" reason="Never" /> -->
+      <disable_collisions link1="${prefix}link7" link2="vader_gripper_base_link" reason="Adjacent" />
+      <disable_collisions link1="${prefix}link_eef" link2="vader_gripper_base_link" reason="Adjacent" />
+      <disable_collisions link1="fing_1" link2="vader_gripper_base_link" reason="Adjacent" />
+      <disable_collisions link1="fing_2" link2="vader_gripper_base_link" reason="Adjacent" />
+      <disable_collisions link1="thumb_1" link2="vader_gripper_base_link" reason="Adjacent" />
+    </xacro:if>
+    <!-- vader cutter -->
+    <xacro:if value="${_use_vader_cutter}">
+      <group name="${prefix}vader_cutter">
+        <!-- <joint name="${prefix}v_cutter_fix" /> -->
+        <link name="blade_stationary" />
+        <link name="blade_moving" />
+        <link name="${prefix}link_tcp" />
+        <link name="vader_cutter_base_link"/>
+      </group>
+      <end_effector name="${prefix}vader_cutter" parent_link="${prefix}link_tcp" group="${prefix}vader_cutter" />
+      <!-- <passive_joint name="${prefix}v_cutter_fix" /> -->
+      <!-- <disable_collisions link1="${prefix}link3" link2="" reason="Never" />
+      <disable_collisions link1="${prefix}link6" link2="${prefix}xarm_vacuum_cutter_link" reason="Never" />
+      <disable_collisions link1="${prefix}link7" link2="${prefix}xarm_vacuum_cutter_link" reason="Never" /> -->
+      <disable_collisions link1="${prefix}link7" link2="vader_cutter_base_link" reason="Adjacent" />
+      <disable_collisions link1="${prefix}link_eef" link2="vader_cutter_base_link" reason="Adjacent" />
+      <disable_collisions link1="blade_stationary" link2="vader_cutter_base_link" reason="Adjacent" />
+      <disable_collisions link1="blade_moving" link2="vader_cutter_base_link" reason="Adjacent" />
+      <disable_collisions link1="blade_moving" link2="blade_stationary" reason="Adjacent" />
+    </xacro:if>
     <!-- other box -->
     <xacro:if value="${_use_other_geometry}">

File: src/xarm_description/srdf/dual_xarm.srdf.xacro (robot description, xacro)
@@ -10,4 +10,8 @@
   <xacro:arg name="add_gripper_1" default="false" />
   <xacro:arg name="add_gripper_2" default="false" />
+  <xacro:arg name="add_vader_gripper_1" default="false" />
+  <xacro:arg name="add_vader_gripper_2" default="false" />
+  <xacro:arg name="add_vader_cutter_1" default="false" />
+  <xacro:arg name="add_vader_cutter_2" default="false" />
   <xacro:arg name="add_vacuum_gripper_1" default="false" />
   <xacro:arg name="add_vacuum_gripper_2" default="false" />
@@ -16,6 +20,8 @@
   <xacro:include filename="$(find xarm_description)/srdf/xarm_macro.srdf.xacro" />
   <xacro:xarm_macro_srdf prefix="$(arg prefix_1)" dof="$(arg dof_1)" robot_type="$(arg robot_type_1)"
+    add_vader_gripper="$(arg add_vader_gripper_1)" add_vader_cutter="$(arg add_vader_cutter_1)"
     add_gripper="$(arg add_gripper_1)" add_vacuum_gripper="$(arg add_vacuum_gripper_1)" add_other_geometry="$(arg add_other_geometry_1)" />
   <xacro:xarm_macro_srdf prefix="$(arg prefix_2)" dof="$(arg dof_2)" robot_type="$(arg robot_type_2)"
+    add_vader_gripper="$(arg add_vader_gripper_2)" add_vader_cutter="$(arg add_vader_cutter_2)"
     add_gripper="$(arg add_gripper_2)" add_vacuum_gripper="$(arg add_vacuum_gripper_2)" add_other_geometry="$(arg add_other_geometry_2)" />
 </robot>

File: src/xarm_description/srdf/xarm.srdf.xacro (robot description, xacro)
@@ -6,8 +6,11 @@
   <xacro:arg name="robot_type" default="xarm" />
   <xacro:arg name="add_gripper" default="false"/>
+  <xacro:arg name="add_vader_gripper" default="false"/>
+  <xacro:arg name="add_vader_cutter" default="false"/>
   <xacro:arg name="add_vacuum_gripper" default="false" />
   <xacro:arg name="add_other_geometry" default="false" />
   <xacro:include filename="$(find xarm_description)/srdf/xarm_macro.srdf.xacro" />
   <xacro:xarm_macro_srdf prefix="$(arg prefix)" dof="$(arg dof)" robot_type="$(arg robot_type)"
+    add_vader_gripper="$(arg add_vader_gripper)" add_vader_cutter="$(arg add_vader_cutter)"
     add_gripper="$(arg add_gripper)" add_vacuum_gripper="$(arg add_vacuum_gripper)" add_other_geometry="$(arg add_other_geometry)" />
 </robot>

File: src/xarm_description/srdf/xarm_macro.srdf.xacro (robot description, xacro)
@@ -2,32 +2,10 @@
 <robot xmlns:xacro="http://wiki.ros.org/xacro" name="xarm_srdf">
   <xacro:macro name="xarm_macro_srdf" params="prefix:='' dof:=7 robot_type:='xarm'
+    add_vader_gripper:='false' add_vader_cutter:='false'
     add_gripper:='false' add_vacuum_gripper:='false' add_other_geometry:='false' ">
-    <xacro:if value="${dof == 5}">
-      <xacro:include filename="$(find xarm_description)/srdf/_xarm5_macro.srdf.xacro" />
-      <xacro:xarm5_macro_srdf prefix="${prefix}"
-        add_gripper="${add_gripper}" add_vacuum_gripper="${add_vacuum_gripper}" add_other_geometry="${add_other_geometry}" />
-    </xacro:if>
-    <xacro:if value="${dof == 6}">
-      <xacro:if value="${robot_type == 'uf850'}">
-        <xacro:include filename="$(find xarm_description)/srdf/_uf850_macro.srdf.xacro" />
-        <xacro:uf850_macro_srdf prefix="${prefix}"
-          add_gripper="${add_gripper}" add_vacuum_gripper="${add_vacuum_gripper}" add_other_geometry="${add_other_geometry}"  />
-      </xacro:if>
-      <xacro:if value="${robot_type == 'lite'}">
-        <xacro:include filename="$(find xarm_description)/srdf/_lite6_macro.srdf.xacro" />
-        <xacro:lite6_macro_srdf prefix="${prefix}"
-          add_gripper="${add_gripper}" add_vacuum_gripper="${add_vacuum_gripper}" add_other_geometry="${add_other_geometry}"  />
-      </xacro:if>
-      <xacro:unless value="${robot_type == 'lite' or robot_type == 'uf850'}">
-        <xacro:include filename="$(find xarm_description)/srdf/_xarm6_macro.srdf.xacro" />
-        <xacro:xarm6_macro_srdf prefix="${prefix}"
-          add_gripper="${add_gripper}" add_vacuum_gripper="${add_vacuum_gripper}" add_other_geometry="${add_other_geometry}"  />
-      </xacro:unless>
-    </xacro:if>
-    <xacro:unless value="${dof == 5 or dof == 6}">
-      <xacro:include filename="$(find xarm_description)/srdf/_xarm7_macro.srdf.xacro" />
-      <xacro:xarm7_macro_srdf prefix="${prefix}"
-        add_gripper="${add_gripper}" add_vacuum_gripper="${add_vacuum_gripper}" add_other_geometry="${add_other_geometry}"  />
-    </xacro:unless>
+    <xacro:include filename="$(find xarm_description)/srdf/_xarm7_macro.srdf.xacro" />
+    <xacro:xarm7_macro_srdf prefix="${prefix}"
+    add_vader_gripper="${add_vader_gripper}" add_vader_cutter="${add_vader_cutter}"
+      add_gripper="${add_gripper}" add_vacuum_gripper="${add_vacuum_gripper}" add_other_geometry="${add_other_geometry}"  />
   </xacro:macro>
 </robot>

Commit message: minor bugfixes

File: src/xarm_description/srdf/_xarm7_macro.srdf.xacro (robot description, xacro)
@@ -9,6 +9,6 @@
   <!-- CHAINS: When a chain is specified, all the links along the chain (including endpoints) are included in the group. Additionally, all the joints that are parents to included links are also included. This means that joints along the chain and the parent joint of the base link are included in the group -->
   <!-- SUBGROUPS: Groups can also be formed by referencing to already defined group names -->
-  <xacro:macro name="xarm7_macro_srdf" params="prefix=''
-    add_gripper='false' add_vader_gripper='false' add_vader_cutter='false' add_vacuum_gripper='false' add_other_geometry='false' ">
+  <xacro:macro name="xarm7_macro_srdf" params="prefix:=''
+    add_gripper:='false' add_vader_gripper:='false' add_vader_cutter:='false' add_vacuum_gripper:='false' add_other_geometry:='false' ">
     <xacro:if value="${add_gripper}">
       <xacro:property name="_use_gripper" value="true"/>
@@ -60,5 +60,5 @@
               <xacro:property name="_use_other_geometry" value="false"/>
               <xacro:property name="_use_no_end_effector" value="true"/>
-              <xacro:property name="_use_vader_gripper" value="true"/>
+              <xacro:property name="_use_vader_gripper" value="false"/>
               <xacro:property name="_use_vader_cutter" value="false"/>
             </xacro:unless>
