Commit message: Added storage bin

File: src/xarm_description/urdf/dual_xarm_device.urdf.xacro (robot description, xacro)
@@ -13,4 +13,5 @@
   <xacro:arg name="add_vader_cutter_1" default="false"/>
   <xacro:arg name="add_vader_cutter_2" default="false"/>
+  <xacro:property name="add_bin" value="true"/>
   <xacro:arg name="add_vacuum_gripper_1" default="false"/>
   <xacro:arg name="add_vacuum_gripper_2" default="false"/>
@@ -68,4 +69,8 @@
   <!-- load xarm device -->
   <xacro:include filename="$(find xarm_description)/urdf/xarm_device_macro.xacro" />
+  <xacro:if value="${add_bin}">
+    <xacro:include filename="$(find xarm_description)/urdf/vader/vader_bin.urdf.xacro"/>
+    <xacro:vader_bin_urdf prefix="" attach_to="world"/>
+  </xacro:if>
   <xacro:xarm_device prefix="$(arg prefix_1)" hw_ns="$(arg hw_ns)" limited="$(arg limited)"
     effort_control="$(arg effort_control)" velocity_control="$(arg velocity_control)"

Commit message: Added horizontal/vertical dual-arm mounting, pretty README pictures

File: src/xarm_description/urdf/dual_xarm_device.urdf.xacro (robot description, xacro)
@@ -14,5 +14,17 @@
   <xacro:arg name="add_vader_cutter_2" default="false"/>
   <xacro:property name="add_bin" value="true"/>
-  <xacro:arg name="bin_xyz" default="0 0 0"/>
+  <xacro:arg name="bin_xyz" default="0 -0.3 0"/>
+  <xacro:arg name="arm_spacing" default="0.5"/>
+  <xacro:arg name="arm_height_horizontal_mount" default="0.5"/>
+  <xacro:arg name="horizontal_mount_arms" default="false"/>
+  <!-- <xacro:property name="arm_pitch" value="0"/> -->
+  <xacro:if value="$(arg horizontal_mount_arms)">
+    <xacro:property name="arm_pitch" value="1.57079633"/>
+    <xacro:property name="arm_height" value="$(arg arm_height_horizontal_mount)"/>
+  </xacro:if>
+  <xacro:unless value="$(arg horizontal_mount_arms)">
+    <xacro:property name="arm_pitch" value="0"/>
+    <xacro:property name="arm_height" value="0"/>
+  </xacro:unless>
   <xacro:arg name="add_vacuum_gripper_1" default="false"/>
   <xacro:arg name="add_vacuum_gripper_2" default="false"/>
@@ -81,5 +93,5 @@
     ros2_control_plugin="$(arg ros2_control_plugin)" robot_type="$(arg robot_type_1)"
     load_gazebo_plugin="false" ros2_control_params="$(arg ros2_control_params)"
-    attach_to="world" attach_xyz="0 0 0" attach_rpy="0 0 0"
+    attach_to="world" attach_xyz="0 0 ${arm_height}" attach_rpy="0 ${arm_pitch} 0"
     add_realsense_d435i="$(arg add_realsense_d435i_1)"
     add_d435i_links="$(arg add_d435i_links_1)"
@@ -101,5 +113,5 @@
     ros2_control_plugin="$(arg ros2_control_plugin)" robot_type="$(arg robot_type_2)"
     load_gazebo_plugin="true" ros2_control_params="$(arg ros2_control_params)"
-    attach_to="world" attach_xyz="0 0.5 0" attach_rpy="0 0 0" create_attach_link="false"
+    attach_to="world" attach_xyz="0 $(arg arm_spacing) ${arm_height}" attach_rpy="0 ${arm_pitch} 0" create_attach_link="false"
     add_realsense_d435i="$(arg add_realsense_d435i_2)"
     add_d435i_links="$(arg add_d435i_links_2)"
